Commit message: use collision meshes as visual mesh, remove copies in visual/ folder

File: fanuc_m20id_support/urdf/m20id35_macro.xacro (robot description, xacro)
@@ -8,5 +8,5 @@
         <origin xyz="0 0 0" rpy="0 0 0"/>
         <geometry>
-          <mesh filename="package://fanuc_m20id_support/meshes/m20id35/visual/base_link.stl"/>
+          <mesh filename="package://fanuc_m20id_support/meshes/m20id35/collision/base_link.stl"/>
         </geometry>
         <xacro:material_fanuc_gray40 />
@@ -23,5 +23,5 @@
         <origin xyz="0 0 0" rpy="0 0 0"/>
         <geometry>
-          <mesh filename="package://fanuc_m20id_support/meshes/m20id35/visual/link_1.stl"/>
+          <mesh filename="package://fanuc_m20id_support/meshes/m20id35/collision/link_1.stl"/>
         </geometry>
         <xacro:material_fanuc_yellow />
@@ -38,5 +38,5 @@
         <origin xyz="-0.055 -0.504510 0" rpy="0 0 0"/>
         <geometry>
-          <mesh filename="package://fanuc_m20id_support/meshes/m20id35/visual/link_2.stl"/>
+          <mesh filename="package://fanuc_m20id_support/meshes/m20id35/collision/link_2.stl"/>
         </geometry>
         <xacro:material_fanuc_yellow />
@@ -53,5 +53,5 @@
         <origin xyz="0.0 -0.40615 0" rpy="0 0 0"/>
         <geometry>
-          <mesh filename="package://fanuc_m20id_support/meshes/m20id35/visual/link_3.stl"/>
+          <mesh filename="package://fanuc_m20id_support/meshes/m20id35/collision/link_3.stl"/>
         </geometry>
         <xacro:material_fanuc_yellow />
@@ -68,5 +68,5 @@
         <origin xyz="0 0 0" rpy="0 0 0"/>
         <geometry>
-          <mesh filename="package://fanuc_m20id_support/meshes/m20id35/visual/link_4.stl"/>
+          <mesh filename="package://fanuc_m20id_support/meshes/m20id35/collision/link_4.stl"/>
         </geometry>
         <xacro:material_fanuc_yellow />
@@ -83,5 +83,5 @@
         <origin xyz="0 0 0" rpy="0 0 0"/>
         <geometry>
-          <mesh filename="package://fanuc_m20id_support/meshes/m20id35/visual/link_5.stl"/>
+          <mesh filename="package://fanuc_m20id_support/meshes/m20id35/collision/link_5.stl"/>
         </geometry>
         <xacro:material_fanuc_yellow />
@@ -98,5 +98,5 @@
         <origin xyz="-0.060 0 0" rpy="0 ${radians(-90)} 0"/>
         <geometry>
-          <mesh filename="package://fanuc_m20id_support/meshes/m20id35/visual/link_6.stl"/>
+          <mesh filename="package://fanuc_m20id_support/meshes/m20id35/collision/link_6.stl"/>
         </geometry>
         <xacro:material_fanuc_black />

Commit message: fix opw/urdf offsets: 890&215mm

File: fanuc_m20id_support/urdf/m20id35_macro.xacro (robot description, xacro)
@@ -132,5 +132,5 @@
     </joint>
     <joint name="${prefix}joint_4" type="revolute">
-      <origin xyz="0.28574 0 0.215" rpy="0 0 0"/>
+      <origin xyz="0 0 0.215" rpy="0 0 0"/>
       <parent link="${prefix}link_3"/>
       <child link="${prefix}link_4"/>
@@ -139,5 +139,5 @@
     </joint>
     <joint name="${prefix}joint_5" type="revolute">
-      <origin xyz="0.6038 0 0" rpy="0 0 0"/>
+      <origin xyz="0.890 0 0" rpy="0 0 0"/>
       <parent link="${prefix}link_4"/>
       <child link="${prefix}link_5"/>

Commit message: update joint limits and velocities from datasheet, update reference document in package.xml

File: fanuc_m20id_support/urdf/m20id35_macro.xacro (robot description, xacro)
@@ -66,5 +66,5 @@
     <link name="${prefix}link_4">
       <visual>
-        <origin xyz="0 0 0" rpy="0 0 0"/>
+        <origin xyz="0.2857 0 0" rpy="0 0 0"/>
         <geometry>
           <mesh filename="package://fanuc_m20id_support/meshes/m20id35/collision/link_4.stl"/>
@@ -73,5 +73,5 @@
       </visual>
       <collision>
-        <origin xyz="0 0 0" rpy="0 0 0"/>
+        <origin xyz="0.2857 0 0" rpy="0 0 0"/>
         <geometry>
           <mesh filename="package://fanuc_m20id_support/meshes/m20id35/collision/link_4.stl"/>
@@ -115,5 +115,5 @@
       <child link="${prefix}link_1"/>
       <axis xyz="0 0 1"/>
-      <limit lower="${radians(-175)}" upper="${radians(175)}" effort="0" velocity="${radians(180)}"/>
+      <limit lower="${radians(-170)}" upper="${radians(170)}" effort="0" velocity="${radians(180)}"/>
     </joint>
     <joint name="${prefix}joint_2" type="revolute">
@@ -122,5 +122,5 @@
       <child link="${prefix}link_2"/>
       <axis xyz="0 1 0"/>
-      <limit lower="${radians(-60)}" upper="${radians(76)}" effort="0" velocity="${radians(90)}"/>
+      <limit lower="${radians(-100)}" upper="${radians(160)}" effort="0" velocity="${radians(180)}"/>
     </joint>
     <joint name="${prefix}joint_3" type="revolute">
@@ -129,5 +129,5 @@
       <child link="${prefix}link_3"/>
       <axis xyz="0 -1 0"/>
-      <limit lower="${radians(-121)}" upper="${radians(180)}" effort="0" velocity="${radians(85)}"/>
+      <limit lower="${radians(-190)}" upper="${radians(268)}" effort="0" velocity="${radians(200)}"/>
     </joint>
     <joint name="${prefix}joint_4" type="revolute">
@@ -136,5 +136,5 @@
       <child link="${prefix}link_4"/>
       <axis xyz="-1 0 0"/>
-      <limit lower="${radians(-200)}" upper="${radians(200)}" effort="0" velocity="${radians(120)}"/>
+      <limit lower="${radians(-200)}" upper="${radians(200)}" effort="0" velocity="${radians(350)}"/>
     </joint>
     <joint name="${prefix}joint_5" type="revolute">
@@ -143,5 +143,5 @@
       <child link="${prefix}link_5"/>
       <axis xyz="0 -1 0"/>
-      <limit lower="${radians(-125)}" upper="${radians(125)}" effort="0" velocity="${radians(120)}"/>
+      <limit lower="${radians(-140)}" upper="${radians(140)}" effort="0" velocity="${radians(350)}"/>
     </joint>
     <joint name="${prefix}joint_6" type="revolute">
@@ -150,5 +150,5 @@
       <child link="${prefix}link_6"/>
       <axis xyz="-1 0 0"/>
-      <limit lower="${radians(-270)}" upper="${radians(270)}" effort="0" velocity="${radians(200)}"/>
+      <limit lower="${radians(-270)}" upper="${radians(270)}" effort="0" velocity="${radians(400)}"/>
     </joint>
     <!-- ROS-Industrial 'base' frame: base_link to Fanuc World Coordinates transform -->
